File: prototype.sch (EAGLE design)
At the start: 15 parts

Commit message: Final Draft of schematic
Parts:
- removed BLUE_LED, GREEN_LED, RED_LED: LAP4-BOTTOM, led:LAP4-BOTTOM
- removed VCC_RES: 1k, SparkFun-Resistors:1KOHM-HORIZ-1/4W-1%
- added MOTOR_LED: BLUE, led:LED5MM
- added RUNNING_LED: GREEN, led:LED5MM
- added STANDBY_LED: RED, led:LED5MM
Connections:
- removed net N$10: MOTOR.1, ON/OFF.O
- removed net N$11: DRIVER.A, MOTOR.2
- new net N$1: DRIVER.C, MOTOR.1, ON/OFF.O
- net GND: now also MOTOR_LED.C; no longer BLUE_LED.C
- net GREEN: now also RUNNING_LED.A; no longer GREEN_LED.A
- net N$4: now also STANDBY_LED.C; no longer RED_LED.C
- net N$5: now also RUNNING_LED.C; no longer GREEN_LED.C
- net N$8: now also MOTOR_LED.A; no longer BLUE_LED.A
- net N$9: now also DRIVER.A, MOTOR.2; no longer DRIVER.C, ON/OFF.P, VCC_RES.2
- net RED: now also STANDBY_LED.A; no longer RED_LED.A
- net VCC: now also ON/OFF.P; no longer VCC_RES.1
Other:
- moved on the sheet: DRIVER, MOSFET, MOTOR, ON/OFF, ULTRASONIC
